File: Badges/RedVillage-Defcon/Schematics/Back/GamePip-Back.kicad_pcb (KiCad board)
At the start: 2 copper layers, 134.9 x 102.4 mm, 7 parts

Commit message: CyberTastic schematic done
Parts:
- removed the G*** at (0.00, 0.00) (x7)
- added G*** (x7): LOGO, LOGO, F.Cu at (0.00, 0.00)
