File: Badges/RedVillage-Defcon/Schematics/Test4/GamePip-Back.kicad_pcb (KiCad board)
At the start: 2 copper layers, 134.9 x 102.4 mm, 61 parts, among them J1 2.8" Display, J10 Conn_01x01, J11 Conn_01x01, J12 Conn_01x01, J13 Conn_02x03_Odd_Even, J14 Conn_01x03, J2 USB_C_Plug_USB2.0, J3 Conn_01x03, J5 Cap Sense, J6 Cap Sense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

Commit message: V1 complete
Parts:
- removed C10, C11: 100nF, Capacitor_SMD:C_0805_2012Metric
- removed J7: Conn_01x02, Connector_PinSocket_2.54mm:PinSocket_1x02_P2.54mm_Vertical
- moved J5 146.3 mm to (201.0, 119.1)
- moved J3 91.2 mm to (169.0, 83.0)
- moved J6 61.9 mm to (88.1, 119.2)
Routing:
- net Net-(J5-Pad1): track 0.00 -> 84.1 mm
- net Disp_RESET: track 0.00 -> 71.6 mm, vias 0 -> 2
- net Net-(J6-Pad1): track 0.00 -> 53.1 mm, vias 0 -> 2
- net WR: track 0.00 -> 45.8 mm
- net RS: track 0.00 -> 44.9 mm
- net DE: track 0.00 -> 43.4 mm
- net XR: track 0.00 -> 39.5 mm, vias 0 -> 2
- net XL: track 0.00 -> 38.6 mm, vias 0 -> 2
- net YD: track 0.00 -> 37.0 mm, vias 0 -> 2
- net YU: track 0.00 -> 36.1 mm, vias 0 -> 2
- net VSS: track 9.76 -> 44.7 mm, vias 0 -> 24
- net VCC: track 273.2 -> 278.8 mm
- net +5V: track 131.5 -> 134.3 mm
- net Net-(SW10-Pad1): track 24.9 -> 26.4 mm
- added copper zone on B.Cu, net VSS
- added copper zone on F.Cu, net VSS
