File: Badges/RedVillage-Defcon/Schematics/Front/GamePip.kicad_pcb (KiCad board)
At the start: 2 copper layers, 134.9 x 105.3 mm, 7 parts

Commit message: Further updates
Parts:
- removed the G*** at (0.00, 0.00) (x7)
- added G*** (x7): LOGO, LOGO, F.Cu at (112.2, 113.1)
Other:
- outline, holes or cut-outs redrawn
- net class Default removed

Commit message: V1 complete
Other:
- board text added: "JLCJLCJLCJLC"
Changed lines of the file:
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@@
   (gr_line (start 84.3231 106.4651) (end 84.4441 106.5747) (layer "Edge.Cuts") (width 0.1))
   (gr_line (start 200.247 69.3878) (end 200.247 69.3878) (layer "Edge.Cuts") (width 0.1))
+  (gr_text "JLCJLCJLCJLC" (at 125.6 103.8) (layer "B.SilkS")
+    (effects (font (size 1.5 1.5) (thickness 0.3)))
+  )
 )
