File: Badges/Defcon32/Schematics/MilkTastic.kicad_sch (KiCad schematic)
At the start: 34 parts, among them J1 2.8" Display, J2 SAO Conn, J3 Conn_01x04, J4 Conn_01x01, J5 XYAB, J7 Conn_01x01, J8 DPad, Q1 Q_NPN_BCE, SW1 LB, SW2 RB, SW7 Start/Sel, SW8 SW_SPDT, U1 MilkV Duo, U2 SK6812_Side, U3 SK6812_Side, U4 SK6812_Side, U5 SK6812_Side

Commit message: Lets panel
Parts:
- added H5, H6: MountingHole, MountingHole:MountingHole_3.2mm_M3, symbol Mechanical:MountingHole
- added J6: Ethernet, Connector_PinHeader_2.54mm:PinHeader_1x05_P2.54mm_Vertical, symbol Connector_Generic:Conn_01x05
- added JP1: USB_Pwr, Jumper:SolderJumper-2_P1.3mm_Open_TrianglePad1.0x1.5mm, symbol Jumper:Jumper_2_Small_Open
- added RN2, RN3, RN4: R_Pack04, Resistor_SMD:R_Array_Convex_4x0603, symbol Device:R_Pack04
- RN1: footprint (none) -> Resistor_SMD:R_Array_Convex_4x0603
- SW1, SW2: footprint UL_Buttons:BZCN-TSC005A_Button -> UE_Buttons:TSB003A3518A_RightAngle_Anchor
- SW7: footprint UL_Buttons:StartSel -> UE_Buttons:StartSel-Dome
- SW8: footprint UL_Buttons:SK-3296S_switch -> UE_Buttons:SK-3296S_switch
- U1: footprint UL_Module:MIlkV-Duo -> UE_Module:MIlkV-Duo
- U2, U3, U4, U5: footprint UL_LED:SK6812SIDE-A-RVS -> UE_LED:SK6812SIDE-A-RVS
Connections:
- net BV is gone; now on net Up: U1.27 (GPIOA26)
- net B: now also U1.4 (GPIOA26), RN3.8 (R1.2)
- net B1: now also D3.4 (BK), U1.7 (GPIOA20); no longer U1.24 (GPIOA22)
- net B2: no longer D3.4 (BK)
- net Down: now also U1.25 (GPIOA25), RN4.7 (R2.2); no longer U1.6 (GPIOA19)
- net G1: now also D3.2 (GK), U1.6 (GPIOA19); no longer U1.25 (GPIOA25)
- net Left: now also U1.26 (GPIOA27), RN4.6 (R3.2); no longer U1.5 (GPIOA25)
- net LeftBumper: now also U1.1 (GPIOA28), RN2.8 (R1.2)
- net R1: now also D3.1 (RK), U1.5 (GPIOA25); no longer U1.26 (GPIOA27)
- net Right: now also U1.24 (GPIOA22), RN4.8 (R1.2); no longer U1.7 (GPIOA20)
- net RightBumper: now also U1.2 (GPIOA29), RN2.7 (R2.2)
- net Select: now also RN2.6 (R3.2)
- net Start: now also RN2.5 (R4.2)
- net Up: now also RN4.5 (R4.2); no longer U1.4 (GPIOA26)
- net VCC: now also J1.36 (Pin_36), U1.35 (3V3_Out), RN2.1 (R1.1), RN2.2 (R2.1), RN2.3 (R3.1), RN2.4 (R4.1), RN3.1 (R1.1), RN3.2 (R2.1), RN3.3 (R3.1), RN3.4 (R4.1), RN4.1 (R1.1), RN4.2 (R2.1), RN4.3 (R3.1), RN4.4 (R4.1); no longer D1.1 (K), U1.39 (VSYS)
- net VSS: no longer U1.43 (VSS)
- net X: now also RN3.5 (R4.2)
- net Y: now also RN3.6 (R3.2)
- net at D3.3 (A): now also RN1.1 (R1.1); no longer RN1.4 (R4.1)
- net at D2.3 (A): now also RN1.4 (R4.1); no longer RN1.1 (R1.1)
- net at U1.40 (VBUS): now also JP1.1 (A)
- net at U1.41 (TX+): now also J6.1 (Pin_1)
- net at U1.42 (TX-): now also J6.2 (Pin_2)
- net at U1.44 (RX+): now also J6.4 (Pin_4)
- net at U1.45 (RX-): now also J6.5 (Pin_5)
- removed net G2: D3.2 (GK), U1.2 (GPIOA29)
- removed net R2: D3.1 (RK), U1.1 (GPIOA28)
- removed net VDD: C5.1, J1.2 (Pin_2), J1.36 (Pin_36), J5.1 (Pin_1), U1.11 (GPIOA21), U1.35 (3V3_Out)
- new net: J6.3 (Pin_3), U1.43 (VSS)
- new net +BATT: C5.1, D1.1 (K), J1.2 (Pin_2), JP1.2 (B), U1.39 (VSYS)
- new net Abtn: J5.1 (Pin_1), RN3.7 (R2.2), U1.11 (GPIOA21)
- no-connect marks 37 -> 36
Other:
- moved on the sheet: BT1, D1, J4, J7, SW8, U1
