File: Badges/Defcon32/Schematics/_autosave-MilkTastic.kicad_sch (KiCad schematic)
At the start: 34 parts, among them J1 2.8" Display, J2 SAO Conn, J3 Conn_01x04, J4 Conn_01x01, J5 XYAB, J7 Conn_01x01, J8 DPad, Q1 Q_NPN_BCE, SW1 LB, SW2 RB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

Commit message: Layout complete
Parts:
- RN1: footprint (none) -> Resistor_SMD:R_Array_Convex_4x0603
- SW1, SW2: footprint UL_Buttons:BZCN-TSC005A_Button -> UE_Buttons:TSB003A3518A_RightAngle_Anchor
- SW7: footprint UL_Buttons:StartSel -> UE_Buttons:StartSel-Dome
- SW8: footprint UL_Buttons:SK-3296S_switch -> UE_Buttons:SK-3296S_switch
- U1: footprint UL_Module:MIlkV-Duo -> UE_Module:MIlkV-Duo
Connections:
- net VCC: now also C5.1, J1.2 (Pin_2), J5.1 (Pin_1), U1.11 (GPIOA21)
- net VDD: no longer C5.1, J1.2 (Pin_2), J5.1 (Pin_1), U1.11 (GPIOA21)
Changed lines of the file:
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@@
 	(paper "A4")
 	(junction
-		(at 115.57 176.53)
-		(diameter 0)
-		(color 0 0 0 0)
-	)
-	(junction
 		(at 256.54 147.32)
 		(diameter 0)
@@
 		(color 0 0 0 0)
 	)
+	(junction
+		(at 115.57 176.53)
+		(diameter 0)
+		(color 0 0 0 0)
+	)
 	(no_connect
 		(at 191.77 110.49)
@@
 	(wire
 		(pts
-			(xy 115.57 176.53) (xy 120.65 176.53)
-		)
-		(stroke
-			(width 0)
-			(type default)
-		)
-	)
-	(wire
-		(pts
 			(xy 273.05 147.32) (xy 271.78 147.32)
 		)
@@
 	(wire
 		(pts
+			(xy 115.57 172.72) (xy 115.57 176.53)
+		)
+		(stroke
+			(width 0)
+			(type default)
+		)
+	)
+	(wire
+		(pts
 			(xy 33.02 189.23) (xy 33.02 191.77)
 		)
@@
 	(wire
 		(pts
+			(xy 115.57 176.53) (xy 120.65 176.53)
+		)
+		(stroke
+			(width 0)
+			(type default)
+		)
+	)
+	(wire
+		(pts
 			(xy 172.72 143.51) (xy 175.26 143.51)
 		)
@@
 	(wire
 		(pts
-			(xy 115.57 176.53) (xy 115.57 181.61)
-		)
-		(stroke
-			(width 0)
-			(type default)
-		)
-	)
-	(wire
-		(pts
 			(xy 29.21 166.37) (xy 38.1 166.37)
 		)
@@
 			)
 		)
-		(property "Footprint" "UL_Buttons:StartSel"
+		(property "Footprint" "UE_Buttons:StartSel-Dome"
 			(at 119.38 31.75 0)
 			(effects
@@
 		)
 		(property "Value" "VCC"
-			(at 223.52 146.05 90)
+			(at 223.52 147.32 0)
 			(effects
 				(font
@@
 			)
 		)
-		(property "Footprint" "UL_Buttons:BZCN-TSC005A_Button"
+		(property "Footprint" "UE_Buttons:TSB003A3518A_RightAngle_Anchor"
 			(at 88.9 30.48 0)
 			(effects
@@
 	)
 	(symbol
-		(lib_id "power:VDD")
-		(at 115.57 181.61 180)
-		(unit 1)
-		(exclude_from_sim no)
-		(in_bom yes)
-		(on_board yes)
-		(dnp no)
-		(fields_autoplaced yes)
-		(property "Reference" "#PWR033"
-			(at 115.57 177.8 0)
-			(effects
-				(font
-					(size 1.27 1.27)
-				)
-				(hide yes)
-			)
-		)
-		(property "Value" "VDD"
-			(at 118.11 182.8799 0)
-			(effects
-				(font
-					(size 1.27 1.27)
-				)
-				(justify right)
-			)
-		)
-		(property "Footprint" ""
-			(at 115.57 181.61 0)
-			(effects
-				(font
-					(size 1.27 1.27)
-				)
-				(hide yes)
-			)
-		)
-		(property "Datasheet" ""
-			(at 115.57 181.61 0)
-			(effects
-				(font
-					(size 1.27 1.27)
-				)
-				(hide yes)
-			)
-		)
-		(property "Description" ""
-			(at 115.57 181.61 0)
-			(effects
-				(font
-					(size 1.27 1.27)
-				)
-				(hide yes)
-			)
-		)
-		(pin "1"
-		)
-		(instances
-			(project "MilkTastic"
-				(path "/625bbc85-a8f8-46d4-9338-e60d5e5e321d"
-					(reference "#PWR033")
-					(unit 1)
-				)
-			)
-		)
-	)
-	(symbol
 		(lib_id "power:VSS")
 		(at 228.6 153.67 180)
@@
 			)
 		)
-		(property "Footprint" "UL_Buttons:BZCN-TSC005A_Button"
+		(property "Footprint" "UE_Buttons:TSB003A3518A_RightAngle_Anchor"
 			(at 88.9 48.26 0)
 			(effects
@@
 			)
 		)
-		(property "Footprint" ""
+		(property "Footprint" "Resistor_SMD:R_Array_Convex_4x0603"
 			(at 186.69 103.505 90)
 			(effects
@@
 	)
 	(symbol
+		(lib_id "power:VCC")
+		(at 115.57 172.72 0)
+		(mirror y)
+		(unit 1)
+		(exclude_from_sim no)
+		(in_bom yes)
+		(on_board yes)
+		(dnp no)
+		(fields_autoplaced yes)
+		(property "Reference" "#PWR017"
+			(at 115.57 176.53 0)
+			(effects
+				(font
+					(size 1.27 1.27)
+				)
+				(hide yes)
+			)
+		)
+		(property "Value" "VCC"
+			(at 115.57 167.64 0)
+			(effects
+				(font
+					(size 1.27 1.27)
+				)
+			)
+		)
+		(property "Footprint" ""
+			(at 115.57 172.72 0)
+			(effects
+				(font
+					(size 1.27 1.27)
+				)
+				(hide yes)
+			)
+		)
+		(property "Datasheet" ""
+			(at 115.57 172.72 0)
+			(effects
+				(font
+					(size 1.27 1.27)
+				)
+				(hide yes)
+			)
+		)
+		(property "Description" ""
+			(at 115.57 172.72 0)
+			(effects
+				(font
+					(size 1.27 1.27)
+				)
+				(hide yes)
+			)
+		)
+		(pin "1"
+		)
+		(instances
+			(project "MilkTastic"
+				(path "/625bbc85-a8f8-46d4-9338-e60d5e5e321d"
+					(reference "#PWR017")
+					(unit 1)
+				)
+			)
+		)
+	)
+	(symbol
 		(lib_id "power:VSS")
 		(at 38.1 100.33 270)
@@
 		)
 		(property "Value" "VCC"
-			(at 198.12 149.86 90)
+			(at 195.326 147.32 0)
 			(effects
 				(font
@@
 			)
 		)
-		(property "Footprint" "UL_Module:MIlkV-Duo"
+		(property "Footprint" "UE_Module:MIlkV-Duo"
 			(at 233.68 39.37 0)
 			(effects
@@
 		)
 		(property "Value" "VCC"
-			(at 251.46 146.05 90)
+			(at 251.206 147.32 0)
 			(effects
 				(font
@@
 			)
 		)
-		(property "Footprint" "UL_Buttons:SK-3296S_switch"
+		(property "Footprint" "UE_Buttons:SK-3296S_switch"
 			(at 39.37 31.75 0)
 			(effects
