File: Badges/Defcon32/Schematics/MilkTastic.kicad_pcb (KiCad board)
At the start: 2 copper layers, 42 parts, among them J1 2.8" Display, J2 SAO Conn, J3 Conn_01x04, J4 Conn_01x08, J5 Conn_01x04, J6 Conn_01x04, J7 Conn_01x01, Q1 Q_NPN_BCE, SW1 Up, SW2 Down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

Commit message: Layout complete
Parts:
- removed C6: 100nF, Capacitor_SMD:C_0805_2012Metric
- removed J6: Conn_01x04, Connector_PinHeader_2.54mm:PinHeader_1x04_P2.54mm_Vertical
- removed R1, R2: R_Small, Resistor_SMD:R_0805_2012Metric
- removed SW3: Left, UL_Buttons:BZCN-TSC005A_Button
- removed SW4: A, UL_Buttons:BZCN-TSC005A_Button
- removed SW5: B, UL_Buttons:BZCN-TSC005A_Button
- removed SW6: Right, UL_Buttons:BZCN-TSC005A_Button
- removed U6: CH32V003FxPx, Package_SO:TSSOP-20_4.4x6.5mm_P0.65mm
- added J8: DPad, UE_Buttons:Xbox_DPad, F.Cu at (102.0, 75.6)
- D2, D3: footprint UL_LED:XL-3227RGB_LED -> UE_LED:XL-3227RGB_LED
- J1: footprint RedVillage:Omron_XF2M-4015-1A_1x40-1MP_P0.5mm_Horizontal -> UE-Connector:Omron_XF2M-4015-1A_1x40-1MP_P0.5mm_Horizontal
- J4: value Conn_01x08 -> Conn_01x01; footprint Connector_PinHeader_2.54mm:PinHeader_1x08_P2.54mm_Vertical -> Connector_PinHeader_2.54mm:PinHeader_1x01_P2.54mm_Vertical
- J5: value Conn_01x04 -> XYAB; footprint Connector_PinHeader_2.54mm:PinHeader_1x04_P2.54mm_Vertical -> UE_Buttons:Xbox_DPad
- SW1: value Up -> LB; footprint UL_Buttons:BZCN-TSC005A_Button -> UE_Buttons:TSB003A3518A_RightAngle_Anchor
- SW2: value Down -> RB; footprint UL_Buttons:BZCN-TSC005A_Button -> UE_Buttons:TSB003A3518A_RightAngle_Anchor
- SW7: footprint UL_Buttons:StartSel -> UE_Buttons:StartSel-Dome
- SW8: footprint UL_Buttons:SK-3296S_switch -> UE_Buttons:SK-3296S_switch
- U1: footprint UL_Module:MIlkV-Duo -> UE_Module:MIlkV-Duo
- moved SW2 130.5 mm to (227.2, 34.8)
- moved H4 107.9 mm to (116.0, 31.8)
- moved RN1 105.5 mm to (217.4, 51.0)
- moved H3 104.7 mm to (208.3, 31.6)
- moved J5 102.8 mm to (222.9, 75.5)
- moved SW1 76.9 mm to (85.4, 34.7)
- moved J7 68.6 mm to (176.0, 82.6)
- moved SW8 63.8 mm to (183.5, 33.9)
- moved U1 62.7 mm to (202.8, 91.2), turned to 180 degrees
- moved D1 60.5 mm to (173.1, 34.2), turned to 180 degrees
- moved H2 60.0 mm to (210.2, 86.1)
- moved J3 51.0 mm to (168.4, 90.8), turned to 90 degrees
- moved H1 48.7 mm to (113.9, 86.2)
- moved J2 41.1 mm to (135.6, 26.0)
- moved U4 36.2 mm to (194.8, 31.0)
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Connections:
- C1 pad 1: VCC -> A
- C2 pad 1: VCC -> A
- C3 pad 1: VCC -> A
- C4 pad 1: VCC -> A
- D1 pad 1: VCC -> A
- J1 pad 36: A -> VDD
- J1 pad 5: VCC -> A
- J1 pad 6: VCC -> A
- J3 pad 1: VCC -> A
- J5 pad 1: Net-(J5-Pin_1) -> A
- J5 pad 2: Net-(J5-Pin_2) -> B
- J5 pad 3: Net-(J5-Pin_3) -> X
- J5 pad 4: Net-(J5-Pin_4) -> Y
- R4 pad 1: VCC -> A
- RN1 pad 1: unconnected-(RN1-R1.1-Pad1) -> Net-(D2-A)
- RN1 pad 3: SDA -> unconnected-(RN1-R3.1-Pad3)
- RN1 pad 4: SCL -> Net-(D3-A)
- RN1 pad 5: VCC -> A
- RN1 pad 6: VCC -> unconnected-(RN1-R3.2-Pad6)
- RN1 pad 8: unconnected-(RN1-R1.2-Pad8) -> A
- SW1 pad 1: Up -> LeftBumper
- SW2 pad 1: Down -> RightBumper
- U1 pad 1: SCL -> R2
- U1 pad 11: Net-(J6-Pin_1) -> A
- U1 pad 12: Net-(J6-Pin_2) -> /SK6812
- U1 pad 14: Net-(J6-Pin_3) -> Start
- U1 pad 15: Net-(J6-Pin_4) -> Select
- U1 pad 19: unconnected-(U1-GPIOA14-Pad19) -> X
- U1 pad 2: SDA -> G2
- U1 pad 20: unconnected-(U1-GPIOA15-Pad20) -> Y
- U1 pad 24: Net-(J4-Pin_8) -> B1
- U1 pad 25: Net-(J4-Pin_7) -> G1
- U1 pad 26: Net-(J4-Pin_6) -> R1
- U1 pad 27: Net-(J4-Pin_5) -> BV
- U1 pad 29: Net-(J4-Pin_4) -> unconnected-(U1-PWR_GPIO4-Pad29)
- U1 pad 30: Net-(J4-Pin_3) -> unconnected-(U1-RUN-Pad30)
- U1 pad 31: Net-(J4-Pin_2) -> Net-(J4-Pin_1)
- U1 pad 32: Net-(J4-Pin_1) -> B2
- U1 pad 35: A -> VDD
- U1 pad 39: VCC -> A
- U1 pad 4: Net-(J5-Pin_1) -> Up
- U1 pad 5: Net-(J5-Pin_2) -> Left
- U1 pad 6: Net-(J5-Pin_3) -> Down
- U1 pad 7: Net-(J5-Pin_4) -> Right
- U2 pad 2: VCC -> A
- U3 pad 2: VCC -> A
- U4 pad 2: VCC -> A
- U5 pad 2: VCC -> A
Other:
- board outline added: 7 x 7 mm

Commit message: Lets panel
Parts:
- added H5: MountingHole, MountingHole:MountingHole_3.2mm_M3, F.Cu at (81.8, 62.8)
- added H6: MountingHole, MountingHole:MountingHole_3.2mm_M3, F.Cu at (234.4, 62.4)
- added J6: Ethernet, Connector_PinHeader_2.54mm:PinHeader_1x05_P2.54mm_Vertical, F.Cu at (186.5, 29.0)
- added JP1: USB_Pwr, Jumper:SolderJumper-2_P1.3mm_Open_TrianglePad1.0x1.5mm, F.Cu at (176.5, 88.7)
- added RN2: R_Pack04, Resistor_SMD:R_Array_Convex_4x0603, F.Cu at (167.2, 85.2)
- added RN3: R_Pack04, Resistor_SMD:R_Array_Convex_4x0603, F.Cu at (230.7, 57.6)
- added RN4: R_Pack04, Resistor_SMD:R_Array_Convex_4x0603, F.Cu at (114.8, 57.1)
- added kibuzzard-6692EF0B: G***, kibuzzard-6692EF0B, B.Cu at (232.0, 46.8)
- added kibuzzard-6692EF2E: G***, kibuzzard-6692EF2E, F.Cu at (171.2, 63.2)
- added kibuzzard-6692EF4B: G***, kibuzzard-6692EF4B, F.Cu at (192.0, 32.0)
- added kibuzzard-6692EF58: G***, kibuzzard-6692EF58, F.Cu at (174.2, 29.4)
- U2, U3, U4, U5: footprint UL_LED:SK6812SIDE-A-RVS -> UE_LED:SK6812SIDE-A-RVS
- moved J3 82.8 mm to (236.0, 42.9), turned to 0 degrees
- moved U3 40.6 mm to (94.8, 56.8)
- moved U4 38.2 mm to (222.6, 57.2)
- moved J4 34.2 mm to (175.8, 63.2)
- moved C3 33.2 mm to (222.4, 54.5)
- moved C2 30.3 mm to (101.7, 52.1)
- moved SW8 12.7 mm to (174.4, 25.1)
- moved C5 9.63 mm to (106.5, 45.5)
- moved D1 9.38 mm to (166.5, 27.5)
- moved J8 7.00 mm to (95.0, 75.6)
- moved H3 5.36 mm to (203.1, 32.9)
- moved SW7 3.91 mm to (149.0, 91.0)
- moved U2 3.51 mm to (101.7, 37.1)
- moved H4 2.42 mm to (113.9, 33.0)
- moved SW1 1.78 mm to (83.6, 34.8)
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Connections:
- C1 pad 1: A -> VCC
- C2 pad 1: A -> VCC
- C3 pad 1: A -> VCC
- C4 pad 1: A -> VCC
- D3 pad 1: R2 -> R1
- D3 pad 2: G2 -> G1
- D3 pad 4: B2 -> B1
- J1 pad 36: VDD -> VCC
- J1 pad 5: A -> VCC
- J1 pad 6: A -> VCC
- J2 pad 1: A -> VCC
- J3 pad 1: A -> VCC
- J5 pad 1: A -> Abtn
- R4 pad 1: A -> VCC
- RN1 pad 1: Net-(D2-A) -> Net-(D3-A)
- RN1 pad 4: Net-(D3-A) -> Net-(D2-A)
- RN1 pad 5: A -> VCC
- RN1 pad 8: A -> VCC
- U1 pad 1: R2 -> LeftBumper
- U1 pad 11: A -> Abtn
- U1 pad 2: G2 -> RightBumper
- U1 pad 24: B1 -> Right
- U1 pad 25: G1 -> Down
- U1 pad 26: R1 -> Left
- U1 pad 27: BV -> Up
- U1 pad 35: VDD -> VCC
- U1 pad 4: Up -> B
- U1 pad 40: unconnected-(U1-VBUS-Pad40) -> Net-(JP1-A)
- U1 pad 41: unconnected-(U1-TX+-Pad41) -> Net-(J6-Pin_1)
- U1 pad 42: unconnected-(U1-TX--Pad42) -> Net-(J6-Pin_2)
- U1 pad 43: VSS -> Net-(J6-Pin_3)
- U1 pad 44: unconnected-(U1-RX+-Pad44) -> Net-(J6-Pin_4)
- U1 pad 45: unconnected-(U1-RX--Pad45) -> Net-(J6-Pin_5)
- U1 pad 46: unconnected-(U1-USB_DM-Pad46) -> Net-(J9-Pin_2)
- U1 pad 47: unconnected-(U1-USB_DP-Pad47) -> Net-(J9-Pin_1)
- U1 pad 5: Left -> R1
- U1 pad 6: Down -> G1
- U1 pad 7: Right -> B1
- U2 pad 2: A -> VCC
- U3 pad 2: A -> VCC
- U4 pad 2: A -> VCC
- U5 pad 2: A -> VCC
Routing:
- net VCC: track 0.00 -> 321.5 mm, vias 0 -> 10
- net B1: track 0.00 -> 184.6 mm, vias 0 -> 4
- net G1: track 0.00 -> 182.2 mm, vias 0 -> 4
- net R1: track 0.00 -> 181.9 mm, vias 0 -> 4
- net LeftBumper: track 0.00 -> 150.1 mm, vias 0 -> 2
- net Net-(U3-Dout): track 0.00 -> 139.7 mm, vias 0 -> 2
- net Net-(D2-A): track 0.00 -> 133.0 mm, vias 0 -> 2
- net A: track 0.00 -> 131.1 mm, vias 0 -> 6
- net Down: track 0.00 -> 122.4 mm
- net Left: track 0.00 -> 117.4 mm, vias 0 -> 2
- net /SK6812: track 0.00 -> 113.9 mm
- net X: track 0.00 -> 112.4 mm, vias 0 -> 2
- net Up: track 0.00 -> 109.0 mm, vias 0 -> 2
- net Right: track 0.00 -> 105.7 mm
- net RightBumper: track 0.00 -> 100.4 mm, vias 0 -> 2
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- added copper zone on B.Cu, net VSS
- added copper zone on F.Cu, net VSS
Other:
- board size 7 x 7 mm -> 189.9 x 85.6 mm
