File: SAO/ZeldaStones/GoronRuby/Schematics/Goron's_Ruby.kicad_pcb (KiCad board)
At the start: 2 copper layers, 37.5 x 36.6 mm, 11 parts, among them J1 Conn_02x03_Odd_Even

Commit message: Generated panel of stones
Parts:
- removed the G*** at (147.2, 107.8) (x4)
- removed Ref**: Val**, NFCBuisness:W
- added C1: C_Small, Capacitor_SMD:C_0805_2012Metric, B.Cu at (151.7, 109.8)
- added G*** (x2): LOGO, LOGO, F.Cu at (147.2, 107.8)
- added U1: CH32V003FxPx, Package_SO:TSSOP-20_4.4x6.5mm_P0.65mm, B.Cu at (147.0, 110.0)
- moved RN1 0.84 mm to (139.4, 113.8), turned to 0 degrees
Connections:
- D2 pad 2: Net-(D2-Pad2) -> Net-(D2-A)
- D8 pad 2: Net-(D8-Pad2) -> Net-(D8-A)
- J1 pad 3: Net-(J1-Pad3) -> SDA
- J1 pad 4: Net-(J1-Pad4) -> SCL
- J1 pad 5: Net-(J1-Pad5) -> SWIO
- J1 pad 6: Net-(J1-Pad6) -> unconnected-(J1-Pin_6-Pad6)
- RN1 pad 1: Net-(D2-Pad2) -> Net-(D8-A)
- RN1 pad 4: Net-(D8-Pad2) -> Net-(D2-A)
- RN1 pad 5: VCC -> A
- RN1 pad 6: VCC -> B
- RN1 pad 7: VCC -> C
- RN1 pad 8: VCC -> D
Routing:
- net Net-(D8-A): track 0.00 -> 49.7 mm
- net Net-(D8-Pad2): track 35.3 -> 0.00 mm
- net SDA: track 0.00 -> 11.0 mm
- net SWIO: track 0.00 -> 10.7 mm
- net D: track 0.00 -> 10.4 mm
- net SCL: track 0.00 -> 9.82 mm, vias 0 -> 2
- net C: track 0.00 -> 9.37 mm
- net VCC: track 8.06 -> 17.4 mm
- net Net-(D6-A): track 21.4 -> 30.7 mm
- net B: track 0.00 -> 8.39 mm
- net Net-(D2-Pad2): track 7.59 -> 0.00 mm
- net A: track 0.00 -> 7.03 mm
- net Net-(D2-A): track 0.00 -> 6.45 mm
- net VSS: track 5.88 -> 9.03 mm, vias 5 -> 11
- added copper zone on F.Cu, net VSS
Other:
- net class Default removed
- board text removed: "Made For Defcon 27"
