File: SAO/ZeldaStones/ZoraSaphire/Schematics/ZoraSapphire.kicad_pcb (KiCad board)
At the start: 2 copper layers, 39.6 x 34.9 mm, 11 parts, among them J1 Conn_02x03_Odd_Even

Commit message: Generated panel of stones
Parts:
- removed the G*** at (151.6, 96.7) (x4)
- added C1: C_Small, Capacitor_SMD:C_0805_2012Metric, B.Cu at (146.7, 94.5)
- added G*** (x2): LOGO, LOGO, F.Cu at (151.6, 96.7)
- added U1: CH32V003FxPx, Package_SO:TSSOP-20_4.4x6.5mm_P0.65mm, B.Cu at (152.0, 97.8)
- moved RN1 6.89 mm to (158.1, 93.5)
Connections:
- J1 pad 3: Net-(J1-Pad3) -> SDA
- J1 pad 4: Net-(J1-Pad4) -> SCL
- J1 pad 5: Net-(J1-Pad5) -> SWIO
- J1 pad 6: Net-(J1-Pad6) -> unconnected-(J1-Pin_6-Pad6)
- RN1 pad 5: VCC -> D
- RN1 pad 6: VCC -> C
- RN1 pad 7: VCC -> B
- RN1 pad 8: VCC -> A
Routing:
- net SCL: track 0.00 -> 17.4 mm
- net SDA: track 0.00 -> 13.4 mm
- net SWIO: track 0.00 -> 7.91 mm
- net Net-(D2-A): track 9.36 -> 16.1 mm
- net D: track 0.00 -> 6.58 mm
- net Net-(D6-A): track 9.64 -> 3.72 mm
- net VCC: track 9.97 -> 15.7 mm
- net C: track 0.00 -> 5.60 mm
- net Net-(D8-A): track 8.74 -> 3.70 mm
- net B: track 0.00 -> 4.62 mm
- net Net-(D4-A): track 10.4 -> 14.5 mm
- net A: track 0.00 -> 3.64 mm
- net VSS: track 0.00 -> 2.87 mm, vias 3 -> 12
- added copper zone on F.Cu, net VSS
Other:
- net class Default removed
- board text removed: "Made for Defcon 27"
