File: SAO/Korok/Schematics/Korok.kicad_sch (KiCad schematic)
At the start: 8 parts, among them J1 Speaker, J2 Debug, J3 Conn_02x03_Odd_Even, SW1 SW_SPDT, U1 CH32V006, U4 W25Q16JVSS

Commit message: Finished korok and toplight
Parts:
- J1: footprint UE_Buzzer:Dragonstate HDR-120632ZA-3P7 -> UE_Buzzer:Fuet-1230
Changed lines of the file:
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@@
 			)
 		)
-		(property "Footprint" "UE_Buzzer:Dragonstate HDR-120632ZA-3P7"
+		(property "Footprint" "UE_Buzzer:Fuet-1230"
 			(at 195.58 105.41 0)
 			(effects
