File: Badges/Defcon33/Schematics/TopLight/NeoSword_Toplight.kicad_pcb (KiCad board)
At the start: 2 copper layers, 13.3 x 20.4 mm, 7 parts, among them J9 Conn_01x03

Commit message: Progress on bsidesdsm
Changed lines of the file:
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@@
 		)
+	)
+	(gr_poly
+		(pts
+			(xy 156.172355 75.113562) (xy 156.172355 92.619832) (xy 148.852543 92.619832) (xy 141.5333 92.619832)
+			(xy 141.5333 78.311041) (xy 144.197013 78.311041) (xy 145.705086 79.898696) (xy 145.705086 92.597663)
+			(xy 146.68451 92.597663) (xy 146.68451 79.507609) (xy 145.55047 78.311041) (xy 148.852543 74.832184)
+			(xy 152.156889 78.311041) (xy 151.020008 79.507609) (xy 151.020008 92.597663) (xy 152 92.597663)
+			(xy 152 79.898696) (xy 153.508072 78.311041) (xy 148.852543 73.409945) (xy 144.197013 78.311041)
+			(xy 141.5333 78.311041) (xy 141.5333 75.113562) (xy 146.102995 70.160169) (xy 148.852543 70.160169)
+			(xy 151.602659 70.160169)
+		)
+		(stroke
+			(width 0)
+			(type solid)
+		)
+		(fill yes)
+		(layer "F.Cu")
+	)
+	(gr_poly
+		(pts
+			(xy 156.119776 75.123682) (xy 156.119776 92.629882) (xy 148.8 92.629882) (xy 141.480224 92.629882)
+			(xy 141.480224 75.123682) (xy 146.05 70.170118) (xy 148.8 70.170118) (xy 151.55 70.170118)
+		)
+		(stroke
+			(width 0)
+			(type solid)
+		)
+		(fill yes)
+		(layer "F.Mask")
 	)
 	(gr_line
@@
 	)
 	(group ""
+		(members "c80b8a01-ebef-437d-9918-dc955414eb36")
+	)
+	(group ""
+		(members "75eb97fd-dc1e-4279-a977-8e47b8196c46")
+	)
+	(group ""
