File: Products/USBCpwr/Schematics/USBCpwr.kicad_pcb (KiCad board)
At the start: 2 copper layers, 60 x 45 mm, 27 parts, among them J1 USB_C_Receptacle, J3 InterUnit Connections, J4 Output Positive, J5 Output Negative, SW1 SW_DIP_x03, U1 CH224K

Commit message: Progress on bsidesdsm
Parts:
- removed kibuzzard-6774292F: G***, kibuzzard-6774292F
- added kibuzzard-6903877E: G***, kibuzzard-6903877E, F.Cu at (100.5, 67.0)
- added kibuzzard-6903A84F: G***, kibuzzard-6903A84F, F.Cu at (110.0, 76.0)
- kibuzzard-67742882, kibuzzard-67742999, kibuzzard-67742A98, kibuzzard-67742AAA, kibuzzard-67742ABC: moved to B.Cu
- moved kibuzzard-67741D43 33.1 mm to (92.8, 72.4)
- moved kibuzzard-67742CFE 21.0 mm to (108.8, 53.0), turned to 90 degrees
- moved SW1 19.5 mm to (100.8, 72.4), turned to 180 degrees
- moved H2 17.0 mm to (123.0, 36.0)
- moved H3 17.0 mm to (123.0, 75.0)
- moved J3 16.6 mm to (119.4, 56.6)
- moved kibuzzard-67742BC8 16.6 mm to (112.6, 41.7)
- moved kibuzzard-67742BCF 16.6 mm to (112.6, 46.7)
- moved kibuzzard-67742BE6 16.6 mm to (112.6, 57.1)
- moved kibuzzard-67742BF7 16.6 mm to (112.5, 51.7)
- moved J1 15.7 mm to (120.6, 67.3)
- moved kibuzzard-67742882 15.3 mm to (108.2, 45.0), turned to 180 degrees
- moved R2 13.3 mm to (116.5, 75.5)
- moved C1 13.2 mm to (116.5, 73.2)
- moved kibuzzard-67742CEC 12.9 mm to (105.2, 35.5)
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Connections:
- SW1 pad 1: CFG1 -> CFG3
- SW1 pad 3: CFG3 -> CFG1
Routing:
- net Output-: track 40.3 -> 20.0 mm
- net VBUS: track 67.8 -> 47.9 mm, vias 2 -> 0
- net CFG1: track 28.3 -> 9.33 mm
- net CFG2: track 32.8 -> 14.5 mm, vias 0 -> 2
- net CFG3: track 32.5 -> 16.7 mm, vias 4 -> 2
- net Output+: track 35.0 -> 21.8 mm
- net VCC: track 25.3 -> 16.7 mm, vias 2 -> 0
- net VSS: track 2.82 -> 8.93 mm, vias 11 -> 3
- net Net-(U1-VBUS): track 3.25 -> 6.91 mm
- net D+: track 9.83 -> 6.30 mm
- net CC1: track 11.1 -> 7.97 mm
- net CC2: track 11.0 -> 8.14 mm
- net D-: track 8.80 -> 7.25 mm
Other:
- board size 60 x 45 mm -> 43 x 45 mm
