File: Products/USBCpwr/Schematics/USBCpwr.kicad_sch (KiCad schematic)
At the start: 14 parts, among them J1 USB_C_Receptacle, J3 InterUnit Connections, J4 Output Positive, J5 Output Negative, SW1 SW_DIP_x03, U1 CH224K

Commit message: Progress on bsidesdsm
Connections:
- net CFG1: now also SW1.3; no longer SW1.1
- net CFG3: now also SW1.1; no longer SW1.3
Changed lines of the file:
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@@
 (kicad_sch
-	(version 20231120)
+	(version 20250114)
 	(generator "eeschema")
-	(generator_version "8.0")
+	(generator_version "9.0")
 	(paper "A4")
 	(junction
@@
 		(lib_id "Switch:SW_DIP_x03")
 		(at 105.41 45.72 0)
+		(mirror x)
 		(unit 1)
 		(exclude_from_sim no)
@@
 		(on_board yes)
 		(dnp no)
-		(fields_autoplaced yes)
 		(property "Reference" "SW1"
-			(at 105.41 35.56 0)
+			(at 105.41 55.88 0)
 			(effects
 				(font
@@
 		)
 		(property "Value" "SW_DIP_x03"
-			(at 105.41 38.1 0)
+			(at 105.41 53.34 0)
 			(effects
 				(font
@@
 		)
 		(property "Footprint" "Button_Switch_SMD:SW_DIP_SPSTx03_Slide_6.7x9.18mm_W6.73mm_P2.54mm_LowProfile_JPin"
-			(at 105.41 48.26 0)
+			(at 105.41 43.18 0)
 			(effects
 				(font
@@
 		)
 		(property "Datasheet" "~"
-			(at 105.41 48.26 0)
+			(at 105.41 43.18 0)
 			(effects
 				(font
@@
 		)
 	)
+	(embedded_fonts no)
 )
