File: Badges/BsidesDSM26/Schematics/BsidesDSM26.kicad_pcb (KiCad board)
At the start: 2 copper layers, 16 parts, among them J1 USB_C_Plug_USB2.0, Q1 PMOS, Q2 PMOS

Commit message: Hard part done save
Parts:
- added AE1: NFC_ANT, UE_Module:NFC Anenna, F.Cu at (153.5, 57.2)
- added AE2: 2.4GHz ANT, RF_Antenna:Texas_SWRA117D_2.4GHz_Left, F.Cu at (155.3, 133.3)
- added BT1: Battery_Cell, UE_Battery:AA_TH, F.Cu at (37.6, 27.7)
- added BZ1: Buzzer, Buzzer_Beeper:Buzzer_CUI_CPT-9019S-SMT, F.Cu at (41.3, 163.7)
- added C10: 100nF, Capacitor_SMD:C_0805_2012Metric, F.Cu at (265.4, 67.3)
- added C11: 30p, Capacitor_SMD:C_0603_1608Metric, F.Cu at (154.4, 99.7)
- added C12: 30p, Capacitor_SMD:C_0603_1608Metric, F.Cu at (149.2, 99.7)
- added C13: 150p, Capacitor_SMD:C_0603_1608Metric, F.Cu at (154.4, 97.8)
- added C14: 150p, Capacitor_SMD:C_0603_1608Metric, F.Cu at (149.2, 97.8)
- added C15: 100nF, Capacitor_SMD:C_0805_2012Metric, F.Cu at (265.4, 70.3)
- added C16: 100nF, Capacitor_SMD:C_0805_2012Metric, F.Cu at (265.4, 73.3)
- added C17: 2.2u, Capacitor_SMD:C_0805_2012Metric, F.Cu at (158.6, 108.5)
- added C18: 4.7u, Capacitor_SMD:C_0805_2012Metric, F.Cu at (162.5, 110.5)
- added C19: 100n, Capacitor_SMD:C_0603_1608Metric, F.Cu at (158.5, 116.5)
- added C20: 1u, Capacitor_SMD:C_0603_1608Metric, F.Cu at (153.2, 119.8)
- added C21: TBD, Capacitor_SMD:C_0603_1608Metric, F.Cu at (156.3, 120.1)
- added C22: TBD, Capacitor_SMD:C_0603_1608Metric, F.Cu at (156.3, 124.9)
- added C7: 10n, Capacitor_SMD:C_0603_1608Metric, F.Cu at (161.5, 101.2)
- added C8: 24p, Capacitor_SMD:C_0603_1608Metric, F.Cu at (155.2, 102.0)
- added C9: 24p, Capacitor_SMD:C_0603_1608Metric, F.Cu at (148.4, 102.0)
- added H1: MountingHole, UE_Standoff:M3ThreadedStandoff, F.Cu at (63.0, 169.0)
- added H2: MountingHole, UE_Standoff:M3ThreadedStandoff, F.Cu at (63.0, 174.5)
- added H3: MountingHole, UE_Standoff:M3ThreadedStandoff, F.Cu at (63.0, 180.0)
- added H4: MountingHole, UE_Standoff:M3ThreadedStandoff, F.Cu at (63.0, 185.5)
- added J2: U.FL, Connector_Coaxial:U.FL_Hirose_U.FL-R-SMT-1_Vertical, F.Cu at (150.9, 126.6)
- added JP1: SolderJumper_2_Bridged, Jumper:SolderJumper-2_P1.3mm_Bridged_RoundedPad1.0x1.5mm, F.Cu at (155.1, 92.0)
- added JP2: SolderJumper_2_Bridged, Jumper:SolderJumper-2_P1.3mm_Bridged_RoundedPad1.0x1.5mm, F.Cu at (148.4, 92.0)
- added L1: 1u, Inductor_SMD:L_0603_1608Metric, F.Cu at (154.6, 107.0)
- added L2: 1u, Inductor_SMD:L_0603_1608Metric, F.Cu at (149.0, 107.0)
- added L3: 10u, Inductor_SMD:L_0805_2012Metric, F.Cu at (158.7, 110.5)
- added L4: TBD, Inductor_SMD:L_0603_1608Metric, F.Cu at (155.5, 122.5)
- added R2: 2k, Resistor_SMD:R_0603_1608Metric, F.Cu at (158.0, 101.2)
- added R3: 2R, Resistor_SMD:R_0603_1608Metric, F.Cu at (155.1, 95.4)
- added R4: 2R, Resistor_SMD:R_0603_1608Metric, F.Cu at (148.4, 95.3)
- added R5: 100k, Resistor_SMD:R_0805_2012Metric, F.Cu at (22.1, 116.0)
- added R6: 0R, Resistor_SMD:R_0603_1608Metric, F.Cu at (154.6, 126.6)
- added R7: 0R, Resistor_SMD:R_0603_1608Metric, F.Cu at (155.3, 129.0)
- added RN2: R_Pack04, Resistor_SMD:R_Array_Convex_4x0603, F.Cu at (278.4, 123.7)
- added SW1: BOOT, UE_Buttons:TS3315A, F.Cu at (143.8, 116.2)
- added SW2: RST, UE_Buttons:TS3315A, F.Cu at (143.8, 111.4)
- added TP1: TestPoint_Small, TestPoint:TestPoint_Pad_D1.0mm, F.Cu at (152.8, 109.0)
- added TP2: TestPoint_Small, TestPoint:TestPoint_Pad_D1.0mm, F.Cu at (150.8, 109.0)
- added TP3: TestPoint_Small, TestPoint:TestPoint_Pad_D1.0mm, F.Cu at (155.5, 118.3)
- added TP4: TestPoint_Small, TestPoint:TestPoint_Pad_D1.0mm, F.Cu at (155.3, 131.6)
- added U1: SK6812_Side, UE_LED:SK6812SIDE-A-RVS, F.Cu at (273.2, 61.9)
- added U2: SK6812_Side, UE_LED:SK6812SIDE-A-RVS, F.Cu at (273.2, 65.0)
- added U3: SK6812_Side, UE_LED:SK6812SIDE-A-RVS, F.Cu at (273.2, 68.0)
- added U4: SK6812_Side, UE_LED:SK6812SIDE-A-RVS, F.Cu at (273.2, 71.0)
- added U5: CH585M, UE_Module:QFN-48-1EP_5x5mm_P0.35mm_EP3.7x3.7mm, F.Cu at (153.2, 114.1)
- added Y1: 32.768kHz, Crystal:Crystal_SMD_3215-2Pin_3.2x1.5mm, F.Cu at (159.8, 114.2)
- added Y2: 32MHz ±10ppm 12pF, Crystal:Crystal_SMD_3225-4Pin_3.2x2.5mm, F.Cu at (149.9, 119.9)
- C1: value 20pF -> 100nF
- C3: value 100nF -> 20pF
- C4: value 100nF -> 10n; footprint Capacitor_SMD:C_0805_2012Metric -> Capacitor_SMD:C_0603_1608Metric
- C5, C6: value 100nF -> 100p; footprint Capacitor_SMD:C_0805_2012Metric -> Capacitor_SMD:C_0603_1608Metric
- R1: value 100k -> 1k; footprint Resistor_SMD:R_0805_2012Metric -> Resistor_SMD:R_0603_1608Metric
- moved RN1 163.5 mm to (37.6, 180.7)
- moved J1 159.9 mm to (40.9, 171.1)
- moved C2 156.9 mm to (31.1, 172.6)
- moved C3 156.9 mm to (31.1, 175.6)
- moved D2 134.8 mm to (270.1, 117.9)
- moved D3 134.8 mm to (270.1, 121.6)
- moved D4 134.8 mm to (270.1, 125.2)
- moved D5 134.8 mm to (270.1, 128.9)
- moved D1 129.7 mm to (34.8, 114.0)
- moved C1 122.1 mm to (265.4, 58.2)
- moved Q1 119.0 mm to (42.9, 113.9)
- moved Q2 119.0 mm to (42.9, 118.3)
- moved C4 38.9 mm to (160.1, 104.0), turned to 90 degrees
- moved C5 34.5 mm to (154.4, 104.5), turned to 180 degrees
- moved R1 32.9 mm to (162.2, 104.0), turned to -90 degrees
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Connections:
- C1 pad 1: /D- -> VCC
- C2 pad 1: /D+ -> /D-
- C3 pad 1: VCC -> /D+
- C4 pad 1: VCC -> /NFCM
- C5 pad 1: VCC -> Net-(C5-Pad1)
- C6 pad 1: VCC -> VSS
- C6 pad 2: VSS -> Net-(C6-Pad2)
- R1 pad 1: +5V -> /NFCI
- R1 pad 2: VSS -> /NFCM
Routing:
- net /NFCI: track 0.00 -> 18.3 mm
- net Net-(U5-VDCIA): track 0.00 -> 14.9 mm, vias 0 -> 2
- net /NFCM: track 0.00 -> 13.3 mm
- net /~{RST}: track 0.00 -> 12.6 mm
- net /~{ISP}: track 0.00 -> 11.1 mm
- net Net-(JP1-B): track 0.00 -> 9.45 mm, vias 0 -> 2
- net Net-(U5-X32MI): track 0.00 -> 8.51 mm
- net Net-(C11-Pad1): track 0.00 -> 7.10 mm
- net Net-(U5-PA10): track 0.00 -> 6.55 mm
- net Net-(U5-ANT): track 0.00 -> 5.49 mm
- net +3V3: track 0.00 -> 5.28 mm
- net Net-(C12-Pad2): track 0.00 -> 5.10 mm
- net /NFC-: track 0.00 -> 4.98 mm
- net Net-(C22-Pad1): track 0.00 -> 4.98 mm
- net /NFC+: track 0.00 -> 4.89 mm
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
Commit message: ORDERED
Parts:
- added C23: C_Small, Capacitor_SMD:C_0805_2012Metric, F.Cu at (137.5, 129.3)
- added C24: C_Small, Capacitor_SMD:C_0805_2012Metric, F.Cu at (126.5, 128.8)
- added J3: Conn_01x02, Connector_PinHeader_1.00mm:PinHeader_1x02_P1.00mm_Vertical, F.Cu at (166.8, 107.5)
- added J4: Conn_01x02, Connector_PinHeader_1.00mm:PinHeader_1x02_P1.00mm_Vertical, F.Cu at (148.4, 115.5)
- added J5: Conn_01x02, Connector_PinHeader_1.00mm:PinHeader_1x02_P1.00mm_Vertical, F.Cu at (147.5, 111.2)
- added J6: Conn_01x02, Connector_PinHeader_1.00mm:PinHeader_1x02_P1.00mm_Vertical, F.Cu at (149.2, 109.7)
- added J7: Conn_01x04, Connector_PinHeader_2.54mm:PinHeader_1x04_P2.54mm_Vertical, F.Cu at (137.1, 123.3)
- added RN3: R_Pack04, Resistor_SMD:R_Array_Convex_4x0603, F.Cu at (175.3, 106.9)
- added SW3: RST, UE_Buttons:TS3315A, F.Cu at (167.8, 116.5)
- added U6: AMS1117-3.3, Package_TO_SOT_SMD:SOT-223-3_TabPin2, F.Cu at (132.2, 127.0)
- added kibuzzard-69CD6EDC: G***, kibuzzard-69CD6EDC, F.Cu at (169.8, 107.0)
- added kibuzzard-69CD78DF: G***, kibuzzard-69CD78DF, B.Cu at (132.2, 119.2)
- added kibuzzard-69CD78FD: G***, kibuzzard-69CD78FD, F.Cu at (143.8, 119.0)
- added kibuzzard-69CD7907: G***, kibuzzard-69CD7907, F.Cu at (143.2, 112.8)
- added kibuzzard-69CD7919: G***, kibuzzard-69CD7919, F.Cu at (173.2, 116.5)
- added kibuzzard-69CD792A: G***, kibuzzard-69CD792A, F.Cu at (131.5, 135.2)
- added kibuzzard-69CD7944: G***, kibuzzard-69CD7944, F.Cu at (132.4, 138.0)
- added kibuzzard-69CD7953: G***, kibuzzard-69CD7953, F.Cu at (125.2, 140.2)
- added kibuzzard-69CD79CB: G***, kibuzzard-69CD79CB, B.Cu at (151.8, 110.2)
- added kibuzzard-69CD7A0E: G***, kibuzzard-69CD7A0E, B.Cu at (144.8, 111.8)
- added kibuzzard-69CD7A3A: G***, kibuzzard-69CD7A3A, B.Cu at (145.8, 115.0)
- BT1: footprint UE_Battery:AA_TH -> Connector_PinHeader_2.54mm:PinHeader_1x02_P2.54mm_Vertical
- H1, H2, H3, H4: moved to B.Cu
- moved BT1 148.7 mm to (146.8, 128.8), turned to 180 degrees
- moved U1 148.1 mm to (129.7, 98.5)
- moved D2 146.7 mm to (124.7, 99.0)
- moved H2 145.5 mm to (184.0, 93.8)
- moved C1 141.3 mm to (130.9, 101.8)
- moved RN2 140.6 mm to (139.1, 105.2), turned to 90 degrees
- moved U2 137.4 mm to (140.0, 98.5)
- moved D3 137.0 mm to (135.0, 99.0)
- moved BZ1 133.1 mm to (168.8, 125.2)
- moved H3 132.8 mm to (183.8, 124.8)
- moved C10 128.6 mm to (141.4, 101.8)
- moved R5 122.2 mm to (143.3, 131.8)
- moved C3 120.8 mm to (133.2, 111.2), turned to 90 degrees
- moved RN1 119.9 mm to (130.8, 105.2), turned to 90 degrees
- moved C2 117.1 mm to (133.3, 115.5), turned to -90 degrees
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Connections:
- BZ1 pad 1: Buz -> /Buzzer
- C17 pad 1: +3V3 -> VCC
- C2 pad 1: /D- -> /UD-
- C3 pad 1: /D+ -> /UD+
- D1 pad 2: +5V -> +3V3
- J1 pad A6: /D+ -> /UD+
- J1 pad A7: /D- -> /UD-
- J1 pad B6: /D+ -> /UD+
- J1 pad B7: /D- -> /UD-
- Q1 pad 1: +5V -> +3V3
- Q2 pad 1: +5V -> +3V3
- R5 pad 1: +5V -> +3V3
- RN1 pad 1: VSS -> Net-(J1-CC2)
- RN1 pad 2: VSS -> Net-(J1-CC1)
- RN1 pad 7: Net-(J1-CC1) -> VSS
- RN1 pad 8: Net-(J1-CC2) -> VSS
- RN2 pad 5: Net-(D5-A) -> unconnected-(RN2-R4.2-Pad5)
- RN2 pad 6: Net-(D4-A) -> unconnected-(RN2-R3.2-Pad6)
- U5 pad 17: /PB7 -> /UART0-TX
- U5 pad 18: /PB6 -> /SK6812
- U5 pad 20: /PB4 -> /UART0-RX
- U5 pad 3: +3V3 -> VCC
- U5 pad 36: /PA4 -> /Buzzer
- U5 pad 37: /PA5 -> /User
- U5 pad 38: /PA6 -> G4
- U5 pad 39: /PA0 -> B4
- U5 pad 40: /PA1 -> R4
- U5 pad 41: /PA2 -> G3
- U5 pad 42: /PA3 -> B3
- U5 pad 43: /PA15 -> R3
Routing:
- net VCC: track 0.00 -> 127.8 mm, vias 0 -> 5
- net Net-(U2-Dout): track 0.00 -> 44.7 mm, vias 0 -> 2
- net G4: track 0.00 -> 38.7 mm
- net B4: track 0.00 -> 38.2 mm
- net R4: track 0.00 -> 37.9 mm, vias 0 -> 2
- net /SK6812: track 0.00 -> 30.2 mm, vias 0 -> 2
- net G3: track 0.00 -> 29.8 mm, vias 0 -> 2
- net B3: track 0.00 -> 28.8 mm, vias 0 -> 2
- net R3: track 0.00 -> 28.5 mm, vias 0 -> 2
- net +5V: track 0.00 -> 28.4 mm, vias 0 -> 2
- net /UD+: track 0.00 -> 27.4 mm, vias 0 -> 2
- net /UD-: track 0.00 -> 27.0 mm
- net +3V3: track 5.28 -> 29.3 mm, vias 0 -> 2
- net /PB0: track 0.00 -> 17.2 mm, vias 0 -> 1
- net /Buzzer: track 0.00 -> 16.1 mm
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- added copper zone on B.Cu, net VSS
- added copper zone on F.Cu, net VSS
Other:
- board outline added: 66.7 x 121 mm
