File: Badges/BsidesDSM26/Schematics/BsidesDSM26.kicad_pcb (KiCad board)
At the start: 2 copper layers, 66.7 x 121 mm, 89 parts, among them J1 USB_C_Plug_USB2.0, J2 U.FL, J3 Conn_01x02, J4 Conn_01x02, J5 Conn_01x02, J6 Conn_01x02, J8 Speaker, J9 Conn_01x03, Q2 PMOS, SW1 BOOT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

Commit message: PCBA
Parts:
- removed D1: D_Schottky, Diode_SMD:D_SOD-123
- added Q1: CJ3405, Package_TO_SOT_SMD:SOT-23, F.Cu at (143.2, 128.6)
- added R5: 100k, Resistor_SMD:R_0805_2012Metric, F.Cu at (139.6, 124.4)
- added TP5: TP, TestPoint:TestPoint_Pad_D1.0mm, F.Cu at (140.4, 127.2)
- C23, C24: value C_Small -> 10uF
- L3: footprint Inductor_SMD:L_0805_2012Metric -> Inductor_SMD:L_1008_2520Metric
- Q2: value PMOS -> CJ3405
- moved Y1 0.92 mm to (159.9, 114.1)
- moved C18 0.67 mm to (162.8, 111.1)
- moved L3 0.62 mm to (158.8, 111.1)
Connections:
- Q2 pad 1: +3V3 -> +5V
- Q2 pad 2: BattPos -> Net-(Q1-S)
Routing:
- net +3V3: track 25.8 -> 12.5 mm, vias 2 -> 0
- net +5V: track 28.4 -> 39.0 mm
- net BattPos: track 45.0 -> 50.7 mm
- net Net-(U5-VDCIA): track 16.8 -> 11.5 mm
- net Net-(Q1-S): track 0.00 -> 4.86 mm
- net VCC: track 166.3 -> 165.2 mm

Commit message: ch585
Parts:
- moved C21 0.20 mm to (156.1, 120.1)
- moved L4 0.20 mm to (155.3, 122.5)
- moved TP3 0.20 mm to (155.3, 118.3)
Connections:
- C24 pad 1: +3V3 -> VCC
- U6 pad 2: +3V3 -> VCC
Routing:
- net VCC: track 165.2 -> 179.6 mm
- net +3V3: track 12.5 -> 0.00 mm
- net Net-(U5-VDCIA): track 11.5 -> 16.7 mm, vias 2 -> 3
- net VSS: vias 144 -> 143
