File: Badges/BsidesDSM26/Schematics/_autosave-BsidesDSM26.kicad_pcb (KiCad board)
At the start: 2 copper layers, 66.7 x 121 mm, 89 parts, among them J1 USB_C_Plug_USB2.0, J2 U.FL, J3 Conn_01x02, J4 Conn_01x02, J5 Conn_01x02, J6 Conn_01x02, J8 Speaker, J9 Conn_01x03, Q2 PMOS, SW1 BOOT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

Commit message: PCBA
Parts:
- added TP5: TestPoint_Small, TestPoint:TestPoint_Pad_D1.0mm, F.Cu at (144.2, 127.0)
Routing:
- net BattPos: track 45.0 -> 47.1 mm
Changed lines of the file:
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@@
 		)
 	)
+	(footprint "TestPoint:TestPoint_Pad_D1.0mm"
+		(layer "F.Cu")
+		(at 144.2 127)
+		(descr "SMD pad as test Point, diameter 1.0mm")
+		(tags "test point SMD pad")
+		(property "Reference" "TP5"
+			(at 0 -1.448 0)
+			(layer "F.SilkS")
+			(effects
+				(font
+					(size 1 1)
+					(thickness 0.15)
+				)
+			)
+		)
+		(property "Value" "TestPoint_Small"
+			(at 0 1.55 0)
+			(layer "F.Fab")
+			(effects
+				(font
+					(size 1 1)
+					(thickness 0.15)
+				)
+			)
+		)
+		(property "Datasheet" "~"
+			(at 0 0 0)
+			(unlocked yes)
+			(layer "F.Fab")
+			(hide yes)
+			(effects
+				(font
+					(size 1.27 1.27)
+					(thickness 0.15)
+				)
+			)
+		)
+		(property "Description" "test point"
+			(at 0 0 0)
+			(unlocked yes)
+			(layer "F.Fab")
+			(hide yes)
+			(effects
+				(font
+					(size 1.27 1.27)
+					(thickness 0.15)
+				)
+			)
+		)
+		(property ki_fp_filters "Pin* Test*")
+		(sheetname "/")
+		(sheetfile "BsidesDSM26.kicad_sch")
+		(attr exclude_from_pos_files)
+		(fp_circle
+			(center 0 0)
+			(end 0 0.7)
+			(stroke
+				(width 0.12)
+				(type solid)
+			)
+			(fill no)
+			(layer "F.SilkS")
+		)
+		(fp_circle
+			(center 0 0)
+			(end 1 0)
+			(stroke
+				(width 0.05)
+				(type solid)
+			)
+			(fill no)
+			(layer "F.CrtYd")
+		)
+		(fp_text user "${REFERENCE}"
+			(at 0 -1.45 0)
+			(layer "F.Fab")
+			(effects
+				(font
+					(size 1 1)
+					(thickness 0.15)
+				)
+			)
+		)
+		(pad "1" smd circle
+			(at 0 0)
+			(size 1 1)
+			(layers "F.Cu" "F.Mask")
+			(net 24 "BattPos")
+			(pinfunction "1")
+			(pintype "passive")
+		)
+		(embedded_fonts no)
+	)
 	(footprint "Capacitor_SMD:C_0603_1608Metric"
 		(layer "F.Cu")
@@
 	)
 	(segment
+		(start 144.2 127)
+		(end 144.2 124.875)
+		(width 0.2)
+		(layer "F.Cu")
+		(net 24)
+	)
+	(segment
 		(start 144.325 125)
 		(end 144.2 124.875)
@@
 	)
 	(segment
-		(start 134 127.25)
-		(end 132.676776 127.25)
+		(start 139.7 128.3)
+		(end 139.9 128.5)
 		(width 0.2)
 		(layer "F.Cu")
@@
 	)
 	(segment
-		(start 139 127.6)
-		(end 139.9 128.5)
+		(start 134 127.25)
+		(end 132.676776 127.25)
 		(width 0.2)
 		(layer "F.Cu")
@@
 	)
 	(segment
-		(start 132.25 127.375)
-		(end 132.25 130.15)
+		(start 139 127.25)
+		(end 139.25 127.25)
 		(width 0.2)
 		(layer "F.Cu")
@@
 	)
 	(segment
-		(start 139 127.25)
-		(end 139 127.6)
+		(start 132.25 127.375)
+		(end 132.25 130.15)
 		(width 0.2)
 		(layer "F.Cu")
@@
 		(width 0.2)
 		(layer "F.Cu")
+		(net 39)
+	)
+	(segment
+		(start 139.25 127.25)
+		(end 139.7 127.7)
+		(width 0.2)
+		(layer "F.Cu")
+		(net 39)
+	)
+	(segment
+		(start 139.7 127.7)
+		(end 139.7 128.3)
+		(width 0.2)
+		(layer "F.Cu")
