File: Badges/BsidesDSM26/Schematics/BsidesDSM26.kicad_sch (KiCad schematic)
At the start: 33 parts, among them J11 USB_C_Plug_USB2.0, U1 CH585F

Commit message: Progress
Parts:
- added BT1: Battery_Cell, symbol Device:Battery_Cell
- added BZ1: Buzzer, symbol Device:Buzzer
- added D5: D_Schottky, Diode_SMD:D_0805_2012Metric, symbol Device:D_Schottky_Small
- added Q1, Q2: PMOS, Package_TO_SOT_SMD:SOT-23, symbol Simulation_SPICE:PMOS
- added R7: 100k, Resistor_SMD:R_0805_2012Metric, symbol Device:R_Small
- added RN2: R_Pack04, symbol Device:R_Pack04
Connections:
- net +5V: now also D5.2 (A), Q1.1 (G), Q2.1 (G), R7.1
- net GND: now also U1.Pad (VSS), RN2.1 (R1.1), RN2.2 (R2.1), RN2.3 (R3.1), RN2.4 (R4.1)
- net VSS: now also BZ1.2 (-), R7.2
- net R2: now reaches D2.1 (R)
- net R2: now also U1.29 (PA14)
- net at D2.2 (A): now also RN2.7 (R2.2)
- net G2: now reaches D2.3 (G)
- net G2: now also U1.28 (PA15)
- net B2: now reaches D2.4 (B)
- net B2: now also U1.27 (PA5)
- net R3: now reaches D3.1 (R)
- net R3: now also U1.26 (PA4)
- net at D3.2 (A): now also RN2.6 (R3.2)
- net G3: now reaches D3.3 (G)
- net G3: now also U1.20 (PB22)
- net B3: now reaches D3.4 (B)
- net B3: now also U1.19 (PB23)
- net R1: now reaches D1.1 (R)
- net R1: now also U1.32 (PA11)
- net at D1.2 (A): now also RN2.8 (R1.2)
- net G1: now reaches D1.3 (G)
- net G1: now also U1.31 (PA12)
- net B1: now reaches D1.4 (B)
- net B1: now also U1.30 (PA13)
- net R4: now reaches D4.1 (R)
- net R4: now also U1.18 (PB4)
- net at D4.2 (A): now also RN2.5 (R4.2)
- net G4: now reaches D4.3 (G)
- net G4: now also U1.17 (PB5)
- net B4: now reaches D4.4 (B)
- net B4: now also U1.16 (PB6)
- net Buz: now reaches U1.10 (PB14)
- net Buz: now also BZ1.1 (+)
- net VCC: now reaches U1.4 (VCC)
- net VCC: now also D5.1 (K), Q2.3 (D)
- new net: Q1.2 (S), Q2.2 (S)
- new net BattPos: Q1.3 (D)
Other:
- moved on the sheet: C1, C10, C11, C2, C3, C4, C5, C6, C7, C8, C9, D1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

Commit message: perhaps?
Parts:
- added C3, C4, C5, C6: 100nF, Capacitor_SMD:C_0805_2012Metric, symbol Device:C_Small
- added U2, U3, U4, U5: SK6812_Side, Bsides22:SK6812_Side, symbol BSides22:SK6812_Side
- renumbered C15 to C1, C6 to C11, C2 to C12, C1 to C13, C11 to C14, C7 to C15, C3 to C16, C5 to C17, C16 to C2, C8 to C7, C9 to C8, C4 to C9, D5 to D1, D1 to D2, D2 to D3, D3 to D4, D4 to D5, H3 to H2, H2 to H3, J11 to J1, R7 to R1, R1 to R3, R3 to R4, R4 to R5, R5 to R7
Connections:
- net BattPos: now also BT1.1 (+)
- net VCC: now also C3.1, C4.1, C5.1, C6.1, U2.2 (VCC), U3.2 (VCC), U4.2 (VCC), U5.2 (VCC)
- net VSS: now also BT1.2 (-), C3.2, C4.2, C5.2, C6.2, U2.4 (GND), U3.4 (GND), U4.4 (GND), U5.4 (GND)
- net SK6812: now reaches U1.14 (PB10)
- net SK6812: now also U2.1 (Din)
- new net: U2.3 (Dout), U3.1 (Din)
- new net: U3.3 (Dout), U4.1 (Din)
- new net: U4.3 (Dout), U5.1 (Din)

Commit message: Something something something git language
Parts:
- added C18: C_Small, Capacitor_SMD:C_0805_2012Metric, symbol Device:C_Small
- added J2: Conn_01x04, Connector_PinHeader_2.54mm:PinHeader_1x04_P2.54mm_Vertical, symbol Connector_Generic:Conn_01x04
- BT1: footprint (none) -> UE_Battery:AA_TH
- BZ1: footprint (none) -> Buzzer_Beeper:Buzzer_CUI_CPT-9019S-SMT
- C10, C11, C12, C13, C14, C15, C16, C17, C7, C8, C9: footprint (none) -> Capacitor_SMD:C_0805_2012Metric
- H1, H2, H3, H4: footprint (none) -> UE_Standoff:M3ThreadedStandoff
- L1, L2: footprint (none) -> Inductor_SMD:L_0805_2012Metric
- R2, R3, R4, R5, R6, R7: footprint (none) -> Resistor_SMD:R_0805_2012Metric
- RN2: footprint (none) -> Resistor_SMD:R_Array_Convex_4x0603
- U1: footprint (none) -> Package_DFN_QFN:QFN-32-1EP_4x4mm_P0.4mm_EP2.9x2.9mm
- U2, U3, U4, U5: footprint Bsides22:SK6812_Side -> UE_LED:SK6812SIDE-A-RVS
Connections:
- net Buz: now also U1.9 (PB15); no longer U1.10 (PB14)
- net GND: no longer C8.2, RN2.1 (R1.1), RN2.2 (R2.1), RN2.3 (R3.1), RN2.4 (R4.1), U1.Pad (VSS)
- net VCC: now also C18.2
- net VSS: now also C8.2, RN2.1 (R1.1), RN2.2 (R2.1), RN2.3 (R3.1), RN2.4 (R4.1), U1.Pad (VSS), C18.1
- net at U1.11 (PB13): now also J2.2 (Pin_2)
- net at U1.12 (PB12): now also J2.3 (Pin_3)
- net at U1.13 (PB11): now also J2.4 (Pin_4)
- new net: J2.1 (Pin_1), U1.10 (PB14)

Commit message: Hard part done save
Parts:
- removed C10: 200pF 2%, Capacitor_SMD:C_0805_2012Metric, symbol Device:C_Small
- removed C15: NC, Capacitor_SMD:C_0805_2012Metric, symbol Device:C_Small
- removed C16: 100pF 2%, Capacitor_SMD:C_0805_2012Metric, symbol Device:C_Small
- removed J2: Conn_01x04, Connector_PinHeader_2.54mm:PinHeader_1x04_P2.54mm_Vertical, symbol Connector_Generic:Conn_01x04
- removed JP1: open, symbol Jumper:Jumper_2_Small_Open
- removed R5: 1Ω(4.7Ω), Resistor_SMD:R_0805_2012Metric, symbol Device:R_Small
- removed U1: CH585F, Package_DFN_QFN:QFN-32-1EP_4x4mm_P0.4mm_EP2.9x2.9mm, symbol UE-uC:Ch585F
- added AE1: NFC_ANT, UE_Module:NFC Anenna, symbol Device:Antenna_Loop
- added AE2: 2.4GHz ANT, RF_Antenna:Texas_SWRA117D_2.4GHz_Left, symbol Device:Antenna_Loop
- added C19: 100n, Capacitor_SMD:C_0603_1608Metric, symbol Device:C_Small
- added C20: 1u, Capacitor_SMD:C_0603_1608Metric, symbol Device:C_Small
- added C21, C22: TBD, Capacitor_SMD:C_0603_1608Metric, symbol Device:C_Small
- added C4: 10n, Capacitor_SMD:C_0603_1608Metric, symbol Device:C_Small
- added C5, C6: 100p, Capacitor_SMD:C_0603_1608Metric, symbol Device:C_Small
- added J2: U.FL, Connector_Coaxial:U.FL_Hirose_U.FL-R-SMT-1_Vertical, symbol Connector:Conn_Coaxial
- added JP1, JP2: SolderJumper_2_Bridged, Jumper:SolderJumper-2_P1.3mm_Bridged_RoundedPad1.0x1.5mm, symbol Jumper:SolderJumper_2_Bridged
- added L3: 10u, Inductor_SMD:L_0805_2012Metric, symbol Device:L_Small
- added L4: TBD, Inductor_SMD:L_0603_1608Metric, symbol Device:L_Small
- added R1: 1k, Resistor_SMD:R_0603_1608Metric, symbol Device:R_Small
- added SW1: BOOT, UE_Buttons:TS3315A, symbol Switch:SW_Push
- added SW2: RST, UE_Buttons:TS3315A, symbol Switch:SW_Push
- added TP1, TP2, TP3, TP4: TestPoint_Small, TestPoint:TestPoint_Pad_D1.0mm, symbol Connector:TestPoint_Small
- added U5: CH585M, UE_Module:QFN-48-1EP_5x5mm_P0.35mm_EP3.7x3.7mm, symbol mhardware:CH585M
- added Y1: 32.768kHz, Crystal:Crystal_SMD_3215-2Pin_3.2x1.5mm, symbol Device:Crystal_Small
- added Y2: 32MHz ±10ppm 12pF, Crystal:Crystal_SMD_3225-4Pin_3.2x2.5mm, symbol Device:Crystal_GND24_Small
- C11: value NC -> 30p; footprint Capacitor_SMD:C_0805_2012Metric -> Capacitor_SMD:C_0603_1608Metric
- C12: value 100pF 2% -> 30p; footprint Capacitor_SMD:C_0805_2012Metric -> Capacitor_SMD:C_0603_1608Metric
- C13: value NC -> 150p; footprint Capacitor_SMD:C_0805_2012Metric -> Capacitor_SMD:C_0603_1608Metric
- C14: value 200pF 2% -> 150p; footprint Capacitor_SMD:C_0805_2012Metric -> Capacitor_SMD:C_0603_1608Metric
- C17: value 100pF 2% -> 2.2u
- C18: value C_Small -> 4.7u
- C7: value 10nF -> 10n; footprint Capacitor_SMD:C_0805_2012Metric -> Capacitor_SMD:C_0603_1608Metric
- C8: value 10nF -> 24p; footprint Capacitor_SMD:C_0805_2012Metric -> Capacitor_SMD:C_0603_1608Metric
- C9: value 30pF 2% -> 24p; footprint Capacitor_SMD:C_0805_2012Metric -> Capacitor_SMD:C_0603_1608Metric
- L1, L2: value 1uH -> 1u; footprint Inductor_SMD:L_0805_2012Metric -> Inductor_SMD:L_0603_1608Metric
- R2: value 1k -> 2k; footprint Resistor_SMD:R_0805_2012Metric -> Resistor_SMD:R_0603_1608Metric
- R3: value 2k -> 2R; footprint Resistor_SMD:R_0805_2012Metric -> Resistor_SMD:R_0603_1608Metric
- R4: value NC -> 2R; footprint Resistor_SMD:R_0805_2012Metric -> Resistor_SMD:R_0603_1608Metric
- R6: value NC -> 0R; footprint Resistor_SMD:R_0805_2012Metric -> Resistor_SMD:R_0603_1608Metric; now not fitted
- R7: value 1Ω(4.7Ω) -> 0R; footprint Resistor_SMD:R_0805_2012Metric -> Resistor_SMD:R_0603_1608Metric
- renumbered C3 to C1, C4 to C10, C5 to C15, C6 to C16, C1 to C2, C2 to C3, H3 to H2, H2 to H3, R1 to R5, U2 to U1, U3 to U2, U4 to U3, U5 to U4
Connections:
- net NFC CTR is gone; now on an unnamed net: R2.2
- net NFC+: now also L1.1, TP1.1, U5.9 (PB17); no longer L1.2
- net NFC-: now also L2.1, TP2.1, U5.10 (PB16); no longer L2.2
- net NFCM: now also C4.1, R1.2, U5.8 (PB8); no longer C8.1, R4.2
- net VCC: no longer C18.2
- net VSS: now also C11.2, C12.1, C13.2, C14.1, C17.2, C18.2, AE2.2, C19.2, C20.2, C21.2, C22.2, C4.2, C5.2, C6.1, J2.2 (Ext), SW1.1, SW2.1, U5.49 (GND), Y2.2 (G), Y2.4 (G); no longer C18.1, C8.2
- net at R6.1, R7.1: now also C22.1, L4.2
- net at C11.1, R3.1: now also C13.1, C8.2; no longer C9.1
- removed net GND: C11.2, C12.2, C14.1, R6.2
- net NFC1: no longer names the net of R4.1
- net NFC1: now also C12.2, C14.2, C9.2; no longer C7.2
- new net: C20.1, U5.33 (VINTA)
- new net: C18.1, C19.1, L3.1, U5.1 (VDCID), U5.35 (VDCIA)
- new net: L3.2, U5.2 (VSW)
- new net: C21.1, L4.1, TP3.1, U5.34 (ANT)
- new net: C6.2, C9.1, L2.2
- new net: AE1.1, JP1.2 (B)
- new net: AE1.2, JP2.2 (B)
- new net: U5.32 (X32MI), Y2.1
- new net: U5.31 (X32MO), Y2.3
- new net: C5.1, C8.1, L1.2
- new net: C7.2, R2.1
- new net: AE2.1, R7.2, TP4.1
- new net: U5.47 (PA11), Y1.1
- new net: U5.48 (PA10), Y1.2
- new net: J2.1 (In), R6.2
- new net +3V3: C17.1, U5.3 (VIO33/VDD33)
- new net ANT+: JP1.1 (A), R3.2
- new net ANT-: JP2.1 (A), R4.2
- new net NFCI: C7.1, R1.1, U5.7 (PB9)
- new net PA0: U5.39 (PA0)
- new net PA1: U5.40 (PA1)
- new net PA12: U5.46 (PA12)
- new net PA13: U5.45 (PA13)
- new net PA14: U5.44 (PA14)
- new net PA15: U5.43 (PA15)
- new net PA2: U5.41 (PA2)
- new net PA3: U5.42 (PA3)
- new net PA4: U5.36 (PA4)
- new net PA5: U5.37 (PA5)
- new net PA6: U5.38 (PA6)
- new net PA7: U5.4 (PA7)
- new net PB0: U5.24 (PB0)
- new net PB1: U5.23 (PB1)
- new net PB18: U5.30 (PB18)
- new net PB19: U5.29 (PB19)
- new net PB2: U5.22 (PB2)
- new net PB20: U5.28 (PB20)
- new net PB21: U5.27 (PB21)
- new net PB3: U5.21 (PB3)
- new net PB4: U5.20 (PB4)
- new net PB5: U5.19 (PB5)
- new net PB6: U5.18 (PB6)
- new net PB7: U5.17 (PB7)
- new net RXD1: U5.5 (PA8)
- new net TCK: U5.11 (PB15)
- new net TIO: U5.12 (PB14)
- new net TXD1: U5.6 (PA9)
- new net UD+: U5.15 (PB11)
- new net UD-: U5.16 (PB10)
- new net UD2+: U5.13 (PB13)
- new net UD2-: U5.14 (PB12)
- new net ~{ISP}: SW1.2, U5.26 (PB22)
- new net ~{RST}: SW2.2, U5.25 (PB23)
Other:
- note added: "10µH DCR≤1Ω I_{sat}≥50mA"
- note added: "Antenna Coil"
- note added: "BLE"
- note added: "EMC Filter"
- note added: "Matching"
- note added: "R3 tuning: +R = Lower RX amplitude (attenuate) -R = Higher RX amplitude (boost)"
- note added: "Z_{diff​}: 50Ω @ 13.56 MHz Q_{factor​}: 20 (nom) / 10-35 (range) L_{ant​}: 1∼2μH"
- note added: "~15.9MHz cutoff"
- note removed: "Pa7 is not exposed on this package find a replacement"
- moved on the sheet: BT1, BZ1, C1, C10, C15, C16, D1, D2, D3, D4, D5, Q1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

Commit message: ORDERED
Parts:
- added C23, C24: C_Small, Capacitor_SMD:C_0805_2012Metric, symbol Device:C_Small
- added J3, J4, J5, J6: Conn_01x02, Connector_PinHeader_1.00mm:PinHeader_1x02_P1.00mm_Vertical, symbol Connector_Generic:Conn_01x02
- added J7: Conn_01x04, Connector_PinHeader_2.54mm:PinHeader_1x04_P2.54mm_Vertical, symbol Connector_Generic:Conn_01x04
- added RN3: R_Pack04, Resistor_SMD:R_Array_Convex_4x0603, symbol Device:R_Pack04
- added SW3: RST, UE_Buttons:TS3315A, symbol Switch:SW_Push
- added U6: AMS1117-3.3, Package_TO_SOT_SMD:SOT-223-3_TabPin2, symbol Regulator_Linear:AMS1117-3.3
- BT1: footprint UE_Battery:AA_TH -> Connector_PinHeader_2.54mm:PinHeader_1x02_P2.54mm_Vertical
Connections:
- net D+ is gone; now on net UD+: C3.1, J1.A6 (D+), J1.B6 (D+)
- net D- is gone; now on net UD-: C2.1, J1.A7 (D-), J1.B7 (D-)
- net PA0 is gone; now on net B4: U5.39 (PA0)
- net PA1 is gone; now on net R4: U5.40 (PA1)
- net PA15 is gone; now on net R3: U5.43 (PA15)
- net PA2 is gone; now on net G3: U5.41 (PA2)
- net PA3 is gone; now on net B3: U5.42 (PA3)
- net PA4 is gone; now on net Buzzer: U5.36 (PA4)
- net PA6 is gone; now on net G4: U5.38 (PA6)
- net PB6 is gone; now on net SK6812: U5.18 (PB6)
- net +3V3: now also D1.2 (A), Q1.1 (G), Q2.1 (G), R5.1, C24.1, U6.2 (VO); no longer C17.1, U5.3 (VIO33/VDD33)
- net +5V: now also C23.1, U6.3 (VI); no longer D1.2 (A), Q1.1 (G), Q2.1 (G), R5.1
- net PB0: now also J7.1 (Pin_1)
- net PB1: now also J7.2 (Pin_2)
- net PB2: now also J7.3 (Pin_3)
- net PB3: now also J7.4 (Pin_4)
- net RXD1: now also J3.1 (Pin_1)
- net TCK: now also J6.1 (Pin_1)
- net TIO: now also J6.2 (Pin_2)
- net TXD1: now also J3.2 (Pin_2)
- net UD2+: now also J5.1 (Pin_1)
- net UD2-: now also J5.2 (Pin_2)
- net VCC: now also C17.1, U5.3 (VIO33/VDD33)
- net VSS: now also RN1.7 (R2.2), RN1.8 (R1.2), C23.2, C24.2, RN3.1 (R1.1), RN3.2 (R2.1), RN3.3 (R3.1), RN3.4 (R4.1), SW3.1, U6.1 (GND); no longer RN1.1 (R1.1), RN1.2 (R2.1)
- net at RN2.5 (R4.2): no longer D5.2 (A)
- net at RN2.6 (R3.2): no longer D4.2 (A)
- net at J1.A5 (CC1): now also RN1.2 (R2.1); no longer RN1.7 (R2.2)
- net at J1.B5 (CC2): now also RN1.1 (R1.1); no longer RN1.8 (R1.2)
- net Buz renamed Buzzer
- net PA5 renamed User
- net User: now also SW3.2
- net PB4 renamed UART0-RX
- net UART0-RX: now also J4.1 (Pin_1)
- net PB7 renamed UART0-TX
- net UART0-TX: now also J4.2 (Pin_2)
- new net: D4.2 (A), RN3.8 (R1.2)
- new net: D5.2 (A), RN3.7 (R2.2)
Other:
- moved on the sheet: BZ1, RN1, RN2

Commit message: Lets build some boards
Parts:
- L1, L2: value 1u -> 1uF
Other:
- note added: "C11/12 are optional"
Changed lines of the file:
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@@
 		)
 	)
+	(text "C11/12 are optional\n"
+		(exclude_from_sim no)
+		(at 73.914 169.164 0)
+		(effects
+			(font
+				(size 1.27 1.27)
+			)
+		)
+	)
 	(text "EMC Filter"
 		(exclude_from_sim no)
@@
 			)
 		)
-		(property "Value" "1u"
+		(property "Value" "1uF"
 			(at 44.45 162.814 90)
 			(effects
@@
 			)
 		)
-		(property "Value" "1u"
+		(property "Value" "1uF"
 			(at 44.45 144.78 90)
 			(effects

Commit message: PCBA
Parts:
- removed BZ1: Buzzer, Buzzer_Beeper:Buzzer_CUI_CPT-9019S-SMT, symbol Device:Buzzer
- removed D2, D3, D4, D5: APFA3010, LED_SMD:LED_Kingbright_APFA3010_3x1.5mm_Horizontal, symbol LED:APFA3010
- removed J7: Conn_01x04, Connector_PinHeader_2.54mm:PinHeader_1x04_P2.54mm_Vertical, symbol Connector_Generic:Conn_01x04
- removed Q1: PMOS, Package_TO_SOT_SMD:SOT-23, symbol Simulation_SPICE:PMOS
- removed RN2, RN3: R_Pack04, Resistor_SMD:R_Array_Convex_4x0603, symbol Device:R_Pack04
- added C25: 1nF, Capacitor_SMD:C_0805_2012Metric, symbol Device:C_Small
- added C26, C29: 1uF, Capacitor_SMD:C_0805_2012Metric, symbol Device:C_Small
- added C27, C28: 100nF, Capacitor_SMD:C_0805_2012Metric, symbol Device:C_Small
- added C30: 4.7nF, Capacitor_SMD:C_0805_2012Metric, symbol Device:C_Small
- added J8: Speaker, Connector_Molex:Molex_PicoBlade_53261-0271_1x02-1MP_P1.25mm_Horizontal, symbol Connector_Generic:Conn_01x02
- added J9: Conn_01x03, Connector_PinHeader_2.54mm:PinHeader_1x03_P2.54mm_Vertical, symbol Connector_Generic:Conn_01x03
- added R10: 1K, Resistor_SMD:R_0805_2012Metric, symbol Device:R_Small
- added R8, R9: 30K, Resistor_SMD:R_0805_2012Metric, symbol Device:R_Small
- added TP5: TestPoint_Small, TestPoint:TestPoint_Pad_D1.0mm, symbol Connector:TestPoint_Small
- added U7: NS4150B, Package_SO:MSOP-8_3x3mm_P0.65mm, symbol UE_Module:NS4150B_amp
- BT1: footprint Connector_PinHeader_2.54mm:PinHeader_1x02_P2.54mm_Vertical -> UE_Battery:Keystone5220_AA
- C17: value 2.2u -> 2.2uF
- D1: footprint Diode_SMD:D_0805_2012Metric -> Diode_SMD:D_SOD-123
- L1, L2: value 1uF -> 1uH
- R5: footprint Resistor_SMD:R_0805_2012Metric -> (none)
Connections:
- net BattPos: now also Q2.2 (S), TP5.1
- net PB1: now also J9.1 (Pin_1)
- net PB2: now also J9.2 (Pin_2)
- net PB3: now also J9.3 (Pin_3)
- net VCC: now also C25.1, C26.1, U7.6 (VCC)
- net VSS: now also C25.2, C26.2, C28.2, C29.2, C30.1, U7.7 (GND)
- net B3: no longer names the net of U5.42 (PA3)
- net B4: no longer names the net of U5.39 (PA0)
- net Buzzer renamed ACtrl
- net ACtrl: now also U7.1 (CTRL)
- net G3: no longer names the net of U5.41 (PA2)
- net G4: no longer names the net of U5.38 (PA6)
- net PB0 renamed A_In
- net A_In: now also R10.1
- net R3: no longer names the net of U5.43 (PA15)
- net R4: no longer names the net of U5.40 (PA1)
- new net: C27.1, C30.2, R10.2
- new net: C27.2, R8.1
- new net: C29.1, U7.2 (Bypass)
- new net: R8.2, U7.3 (INP)
- new net: C28.1, R9.1
- new net: R9.2, U7.4 (INN)
- new net: J8.1 (Pin_1), U7.8 (VoP)
- new net: J8.2 (Pin_2), U7.5 (VoN)

Commit message: PCBA
Parts:
- removed D1: D_Schottky, Diode_SMD:D_SOD-123, symbol Device:D_Schottky_Small
- added Q1: CJ3405, Package_TO_SOT_SMD:SOT-23, symbol Simulation_SPICE:PMOS
- C23, C24: value C_Small -> 10uF
- L3: footprint Inductor_SMD:L_0805_2012Metric -> Inductor_SMD:L_1008_2520Metric
- Q2: value PMOS -> CJ3405
- R5: footprint (none) -> Resistor_SMD:R_0805_2012Metric
- TP5: value TestPoint_Small -> TP
Connections:
- net +3V3: no longer Q2.1 (G), R5.1
- net +5V: now also Q2.1 (G), R5.1
- net BattPos: now also Q1.3 (D); no longer Q2.2 (S)
- net VSS: now also Q1.1 (G)
- new net: Q1.2 (S), Q2.2 (S)
Other:
- moved on the sheet: R5, TP5
